File: KiCad/LocoBridge.kicad_pcb (KiCad board)
At the start: 2 copper layers, 85 x 56 mm, 49 parts, among them J1 Conn_01x17_Female, J2 Conn_01x17_Female, J3 RJ12, J4 Conn_01x04_Female, J5 Conn_01x02_Male, Q1 2N3904, Q2 2N3906, Q3 2N3904, U1 LM311, U2 LM2574N-5

Commit message: Updated circuit and board design to improve LN TX reliability
Parts:
- added R9: 1kR, Resistor_THT:R_Axial_DIN0207_L6.3mm_D2.5mm_P7.62mm_Horizontal, F.Cu at (165.3, 109.9)
- R7: value 4k7R -> 2k2R
- R8: value 1kR -> 620R
- R_PMODE1: value 10kR -> 22kR
- moved Q1 5.12 mm to (167.8, 103.5)
- moved R8 2.54 mm to (155.1, 104.8)
- renumbered R9 to R10, R10 to R11, R11 to R12, R12 to R13
Connections:
- net Net-(Q1-Pad2) renamed /LN_TX_1V5
Routing:
- net GND1: track 26.2 -> 21.6 mm
- net /LN_TX_1V5: track 4.45 -> 8.76 mm
- net /LN: track 92.2 -> 90.9 mm
- net /LN_TX: track 8.67 -> 7.62 mm
Other:
- board text added: "LocoBridge for Arduino Micro Board V2"
- board text removed: "LocoBridge for Arduino Micro Board V1"
