File: KiCad/LNGateway.kicad_pcb (KiCad board)
At the start: 2 copper layers, 85 x 56 mm, 50 parts, among them J1 Conn_01x17_Female, J2 Conn_01x17_Female, J3 RJ12, J4 Conn_01x04_Female, J5 Conn_01x02_Male, Q1 2N3904, Q2 2N3906, Q3 2N3904, U1 LM311, U2 LM2574N-5

Commit message: Updated board silk screen for new name
Other:
- board text added: "LNGateway for Arduino Micro Board V2"
- board text removed: "LocoBridge for Arduino Micro Board V2"

Commit message: Added reference to github repo
Other:
- board text added: "Arduino software and circuit documentation: orvio.github.io/LNGateway"
